Commit message: New Changes

File: description/robot.urdf.xacro (robot description, xacro)
@@ -2,3 +2,7 @@
 <robot xmlns:xacro="http://www.ros.org/wiki/xacro"  name="robot">
     <xacro:include filename="robot_core.xacro" />
+    <xacro:include filename="gazebo_control.xacro" />
+    <!-- <xacro:include filename="depth_camera.xacro" />  -->
+    <xacro:include filename="camera.xacro" />
+    <xacro:include filename="lidar.xacro" />
 </robot>

File: description/robot_core.xacro (robot description, xacro)
@@ -14,4 +14,10 @@
         <color rgba="0 1 0 1" />
     </material>
+    <material name="red">
+        <color rgba="1 0 0 1" />
+    </material>
+    <material name="grey">
+        <color rgba="0.5 0.5 0.5 1" />
+    </material>
     <material name="black">
         <color rgba="0 0 0 1" />
@@ -19,4 +25,5 @@
     <!-- BASE LINK  -->
     <link name="base_link">
+        <static>true</static>
     </link>
     <!-- CHASSIS LINK -->
@@ -40,8 +47,11 @@
             </geometry>
         </collision>
-        <xacro:inertial_box mass="6" x="0.4" y="0.25" z="0.18" >
+        <xacro:inertial_box mass="5" x="0.4" y="0.25" z="0.18" >
             <origin xyz="0.2 0.125 0.09" rpy="0 0 0" />
         </xacro:inertial_box>
     </link>
+    <gazebo reference="chassis" >
+        <material>Gazebo/White</material>
+    </gazebo>
     <!-- LEFT FRONT WHEEL LINK -->
     <joint name="left_front_wheel_joint" type="continuous" >
@@ -63,5 +73,13 @@
             </geometry>
         </collision>
+        <xacro:inertial_cylinder mass="0.1" length="0.045" radius="0.55" >
+            <origin xyz="0 0 0" rpy="0 0 0" />
+        </xacro:inertial_cylinder>
     </link>
+    <gazebo reference="left_front_wheel" >
+        <material>Gazebo/Green</material>
+        <mu1 value="0.01" />
+        <mu2 value="0.01" />
+    </gazebo>
     <!-- LEFT BACK WHEEL LINK -->
     <joint name="left_back_wheel_joint" type="continuous" >
@@ -83,5 +101,11 @@
             </geometry>
         </collision>
+        <xacro:inertial_cylinder mass="0.1" length="0.045" radius="0.55" >
+            <origin xyz="0 0 0" rpy="0 0 0" />
+        </xacro:inertial_cylinder>
     </link>
+    <gazebo reference="left_back_wheel" >
+        <material>Gazebo/Blue</material>
+     </gazebo>
     <!-- RIGHT FRONT WHEEL LINK -->
     <joint name="right_front_wheel_joint" type="continuous" >
@@ -103,5 +127,13 @@
             </geometry>
         </collision>
+        <xacro:inertial_cylinder mass="0.1" length="0.045" radius="0.55" >
+            <origin xyz="0 0 0" rpy="0 0 0" />
+        </xacro:inertial_cylinder>
     </link>
+    <gazebo reference="right_front_wheel" >
+        <material>Gazebo/Green</material>
+        <mu1 value="0.01" />
+        <mu2 value="0.01" />
+    </gazebo>
     <!-- RIGHT BACK WHEEL LINK -->
     <joint name="right_back_wheel_joint" type="continuous" >
@@ -123,4 +155,10 @@
             </geometry>
         </collision>
+        <xacro:inertial_cylinder mass="0.1" length="0.045" radius="0.55" >
+            <origin xyz="0 0 0" rpy="0 0 0" />
+        </xacro:inertial_cylinder>
     </link>
+    <gazebo reference="right_back_wheel" >
+        <material>Gazebo/Blue</material>
+    </gazebo>
 </robot>
